Commit message: Minor urdf change.

File: urdf/xacro_include/leg_macro.xacro (robot description, xacro)
@@ -62,5 +62,5 @@
         <mesh filename="package://hexapod_sim/meshes/tibia.dae"/>
       </geometry>
-        <origin xyz="0 -0.02725 0" rpy="${-pi}16 -0.235 0"/>
+        <origin xyz="0 -0.02725 0" rpy="${pi} -0.235 0"/>
       </visual>
       <collision>
