Commit message: Cleanup and first step (robot model, IK and action server).

File: urdf/hexapod.urdf.xacro (robot description, xacro)
@@ -40,5 +40,5 @@
   <joint name="jl11" type="revolute">
     <axis xyz="1 0 0"/>
-    <origin xyz="-0.09 -0.0535 -0.00075" rpy="2.355 ${pi/2} 0"/>
+    <origin xyz="-0.09 -0.0535 -0.00075" rpy="${3*pi/4} ${pi/2} 0"/>
     <parent link="base"/>
     <child link="coxal1"/>
@@ -64,5 +64,5 @@
   <joint name="jl41" type="revolute">
     <axis xyz="1 0 0"/>
-    <origin xyz="-0.09 0.0535 -0.00075" rpy="-2.355 ${pi/2} 0"/>
+    <origin xyz="-0.09 0.0535 -0.00075" rpy="-${3*pi/4} ${pi/2} 0"/>
     <parent link="base"/>
     <child link="coxal4"/>

Commit message: Changed speed and started building fast gait.

File: urdf/hexapod.urdf.xacro (robot description, xacro)
@@ -43,5 +43,5 @@
     <parent link="base"/>
     <child link="coxal1"/>
-    <limit effort="1000.0" lower="${-pi}" upper="${pi}" velocity="${pi/2}"/>
+    <limit effort="1000.0" lower="${-pi}" upper="${pi}" velocity="${2*pi}"/>
     <dynamics damping="0.0" friction="0.0"/>
   </joint>
@@ -51,5 +51,5 @@
     <parent link="base"/>
     <child link="coxal2"/>
-    <limit effort="1000.0" lower="${-pi}" upper="${pi}" velocity="${pi/2}"/>
+    <limit effort="1000.0" lower="${-pi}" upper="${pi}" velocity="${2*pi}"/>
     <dynamics damping="0.0" friction="0.0"/>
   </joint>
@@ -59,5 +59,5 @@
     <parent link="base"/>
     <child link="coxal3"/>
-    <limit effort="1000.0" lower="${-pi}" upper="${pi}" velocity="${pi/2}"/>
+    <limit effort="1000.0" lower="${-pi}" upper="${pi}" velocity="${2*pi}"/>
     <dynamics damping="0.0" friction="0.0"/>
   </joint>
@@ -67,5 +67,5 @@
     <parent link="base"/>
     <child link="coxal4"/>
-    <limit effort="1000.0" lower="${-pi}" upper="${pi}" velocity="${pi/2}"/>
+    <limit effort="1000.0" lower="${-pi}" upper="${pi}" velocity="${2*pi}"/>
     <dynamics damping="0.0" friction="0.0"/>
   </joint>
@@ -75,5 +75,5 @@
     <parent link="base"/>
     <child link="coxal5"/>
-    <limit effort="1000.0" lower="${-pi}" upper="${pi}" velocity="${pi/2}"/>
+    <limit effort="1000.0" lower="${-pi}" upper="${pi}" velocity="${2*pi}"/>
     <dynamics damping="0.0" friction="0.0"/>
   </joint>
@@ -83,5 +83,5 @@
     <parent link="base"/>
     <child link="coxal6"/>
-    <limit effort="1000.0" lower="${-pi}" upper="${pi}" velocity="${pi/2}"/>
+    <limit effort="1000.0" lower="${-pi}" upper="${pi}" velocity="${2*pi}"/>
     <dynamics damping="0.0" friction="0.0"/>
   </joint>

File: urdf/xacro_include/leg_macro.xacro (robot description, xacro)
@@ -26,5 +26,5 @@
       <parent link="coxa${leg_id}"/>
       <child link="femur${leg_id}"/>
-      <limit effort="1000.0" lower="${-pi}" upper="${pi}" velocity="${pi/2}"/>
+      <limit effort="1000.0" lower="${-pi}" upper="${pi}" velocity="${2*pi}"/>
       <dynamics damping="0.0" friction="0.0"/>
     </joint>
@@ -53,5 +53,5 @@
       <parent link="femur${leg_id}"/>
       <child link="tibia${leg_id}"/>
-      <limit effort="1000.0" lower="${-pi}" upper="${pi}" velocity="${pi/2}"/>
+      <limit effort="1000.0" lower="${-pi}" upper="${pi}" velocity="${2*pi}"/>
       <dynamics damping="0.0" friction="0.0"/>
     </joint>
